Commit message: finished implementing bullet bolt 3d env

File: python/py_bullet_env/terrains/stairs.urdf (robot description, URDF)
Before this commit: robot stairs, 4 links, 3 joints
Links:
- link first_step_link: geometry collision box size=0.2 1.0 .1; visual box size=0.2 1.0 .1
- link ground_link: geometry collision box size=.2 1.0 .05; visual box size=.2 1.0 .05
- link second_step_link: geometry collision box size=0.2 1.0 .12; visual box size=0.2 1.0 .12
