Commit message: got steppepper to work in 3d for 5cm ht with push

File: python/py_bullet_env/terrains/plates.urdf (robot description, URDF)
Before this commit: robot stairs, 4 links, 3 joints
Links:
- link first_step_link: geometry collision box size=0.4 1.0 .05; visual box size=0.2 1.0 .05
- link second_step_link: geometry collision box size=0.2 .5 .05; visual box size=0.2 .5 .05
- link third_step_link: geometry collision box size=0.2 0.5 .05; visual box size=0.2 0.5 .05

File: python/py_bullet_env/terrains/stairs.urdf (robot description, URDF)
Before this commit: robot stairs, 4 links, 3 joints
Links:
- added link fourth_step_link, mass .0; collision box size=0.3 1.0 .02; visual box size=0.3 1.0 .02
- link first_step_link: geometry collision box size=0.3 10.0 .08; visual box size=0.3 1.0 .08
- link ground_link: geometry collision box size=.6 1.0 .05; visual box size=.6 1.0 .05
- link second_step_link: geometry collision box size=0.2 .5 .06; visual box size=0.2 .5 .06
- link third_step_link: geometry collision box size=0.2 0.5 .06; visual box size=0.2 0.5 .06
Joints:
- removed joint second_to_third_step
- added joint first_to_fourth_step: type fixed, parent first_step_link, child fourth_step_link, origin xyz=0 0 0 
- added joint first_to_third_step: type fixed, parent first_step_link, child third_step_link, origin xyz=0 0 0 
