Commit message: finished demos for walking along with plots & videos

File: python/py_bullet_env/terrains/push.urdf (robot description, URDF)
Before this commit: robot uneven, 11 links, 10 joints
Links:
- removed link end_step_link
- removed link sixth_step_link
- added link eleventh_step_link, mass .0; collision sphere radius=0.25; visual sphere radius=0.25
- added link tenth_step_link, mass .0; collision sphere radius=0.25; visual sphere radius=0.25
- link ninth_step_link: geometry collision sphere radius=0.25; visual sphere radius=0.25
Joints:
- removed joint eight_to_ninth_step
- removed joint end_joint
- removed joint fifth_to_sixth_step
- added joint ground_to_eleventh_step: type fixed, parent ground_link, child eleventh_step_link, origin xyz=0 0 0 
- added joint ground_to_ninth_step: type fixed, parent ground_link, child ninth_step_link, origin xyz=0 0 0 
- added joint ground_to_tenth_step: type fixed, parent ground_link, child tenth_step_link, origin xyz=0 0 0 
- joint sixth_to_seventh_step: parent sixth_step_link -> ground_link

File: python/py_bullet_env/terrains/stairs.urdf (robot description, URDF)
Before this commit: robot stairs, 5 links, 4 joints
Links:
- added link eight_step_link, mass .0; collision cylinder length=0.4 radius=0.5; visual cylinder length=0.4 radius=0.5
- added link end_step_link, mass .0; collision box size=0.4 0.8 .04; visual box size=0.4 0.8 .04
- added link fifth_step_link, mass .0; collision box size=0.2 0.5 .04; visual box size=0.2 0.5 .04
- added link ninth_step_link, mass .0; collision cylinder length=0.4 radius=0.4; visual cylinder length=0.4 radius=0.4
- added link seventh_step_link, mass .0; collision cylinder length=0.3 radius=0.2; visual cylinder length=0.3 radius=0.2
- added link sixth_step_link, mass .0; collision cylinder length=0.4 radius=0.1; visual cylinder length=0.4 radius=0.1
- link first_step_link: geometry collision box size=0.2 0.2 .04; visual box size=0.2 0.2 .04
- link fourth_step_link: geometry collision box size=0.1 0.5 .02; visual box size=0.12 0.5 .02
- link second_step_link: geometry collision box size=0.2 .2 .04; visual box size=0.2 .2 .04
- link third_step_link: geometry collision box size=0.1 0.4 .06; visual box size=0.1 0.4 .06
Joints:
- added joint first_to_eight_step: type fixed, parent first_step_link, child eight_step_link, origin xyz=0 0 0 
- added joint first_to_end_step: type fixed, parent first_step_link, child end_step_link, origin xyz=0 0 0 
- added joint first_to_fifth_step: type fixed, parent first_step_link, child fifth_step_link, origin xyz=0 0 0 
- added joint first_to_ninth_step: type fixed, parent first_step_link, child ninth_step_link, origin xyz=0 0 0 
- added joint first_to_seventh_step: type fixed, parent first_step_link, child seventh_step_link, origin xyz=0 0 0 
- added joint first_to_sixth_step: type fixed, parent first_step_link, child sixth_step_link, origin xyz=0 0 0 
