Commit message: started working on uneven terrain walking demo

File: python/py_bullet_env/terrains/uneven.urdf (robot description, URDF)
Before this commit: robot stairs, 5 links, 4 joints
Links:
- added link eight_step_link, mass .0; collision sphere radius=0.26; visual sphere radius=0.26
- added link end_link, mass .0; collision box size=.2 0.8 .01; visual box size=.2 0.8 .01
- added link fifth_step_link, mass .0; collision sphere radius=0.2; visual sphere radius=0.2
- added link ninth_step_link, mass .0; collision box size=0.6 0.75 .01; visual box size=0.6 0.75 .01
- added link seventh_step_link, mass .0; collision sphere radius=0.24; visual sphere radius=0.24
- added link sixth_step_link, mass .0; collision box size=.6 0.7 .01; visual box size=.6 0.7 .01
- link first_step_link: geometry collision sphere radius=0.17; visual sphere radius=0.17
- link fourth_step_link: geometry collision sphere radius=0.3; visual sphere radius=0.3
- link ground_link: geometry collision box size=.2 0.8 .01; visual box size=.2 0.8 .01
- link second_step_link: geometry collision sphere radius=0.3; visual sphere radius=0.3
- link third_step_link: geometry collision sphere radius=0.3; visual sphere radius=0.3
Joints:
- added joint eight_to_ninth_step: type fixed, parent eight_step_link, child ninth_step_link, origin xyz=0 0 0 
- added joint fifth_to_sixth_step: type fixed, parent fifth_step_link, child sixth_step_link, origin xyz=0 0 0 
- added joint fourth_to_fifth_step: type fixed, parent fourth_step_link, child fifth_step_link, origin xyz=0 0 0 
- added joint ninth_to_end_step: type fixed, parent ninth_step_link, child end_link
- added joint seventh_to_eight_step: type fixed, parent seventh_step_link, child eight_step_link, origin xyz=0 0 0 
- added joint sixth_to_seventh_step: type fixed, parent sixth_step_link, child seventh_step_link, origin xyz=0 0 0 

Commit message: updated uneven terrain urdf

File: python/py_bullet_env/terrains/uneven.urdf (robot description, URDF)
Before this commit: robot uneven, 11 links, 10 joints
Links:
- removed link end_link
Joints:
- removed joint ninth_to_end_step

Commit message: added captureability analysis demo

File: python/py_bullet_env/terrains/uneven.urdf (robot description, URDF)
Before this commit: robot uneven, 11 links, 10 joints
Links:
- removed link eight_step_link
- removed link fifth_step_link
- removed link ground_link
- removed link seventh_step_link
- added link ground_step_link, mass .0; collision box size=.2 0.8 .01; visual box size=.2 0.8 .01
- link end_step_link: geometry collision box size=0.6 0.5 .01; visual box size=0.6 0.5 .01
- link first_step_link: geometry collision box size=0.3 0.8 .01; visual box size=0.3 0.8 .01
- link fourth_step_link: geometry collision box size=.3 1.4 .01; visual box size=.3 1.4 .01
- link ninth_step_link: geometry collision box size=0.3 1.6 .01; visual box size=0.3 1.6 .01
- link second_step_link: geometry collision box size=0.3 1.2 .01; visual box size=0.3 1.2 .01
- link sixth_step_link: geometry collision box size=.3 0.7 .01; visual box size=.3 0.7 .01
- link third_step_link: geometry collision box size=.3 0.8 .01; visual box size=.3 0.6 .01
Joints:
- removed joint eight_to_ninth_step
- removed joint fifth_to_sixth_step
- removed joint first_to_second_step
- removed joint fourth_to_fifth_step
- removed joint second_to_third_step
- removed joint seventh_to_eight_step
- removed joint sixth_to_seventh_step
- removed joint third_to_fourth_step
- added joint ground_to_fourth_step: type fixed, parent ground_step_link, child fourth_step_link, origin xyz=0 0 0 
- added joint ground_to_ninth_step: type fixed, parent ground_step_link, child ninth_step_link, origin xyz=0 0 0 
- added joint ground_to_second_step: type fixed, parent ground_step_link, child second_step_link, origin xyz=0 0 0 
- added joint ground_to_sixth_step: type fixed, parent ground_step_link, child sixth_step_link, origin xyz=0 0 0 
- added joint ground_to_third_step: type fixed, parent ground_step_link, child third_step_link, origin xyz=0 0 0 
- joint end_joint: parent seventh_step_link -> ground_step_link
- joint ground_to_first_step: origin (none) -> xyz=0 0 0 ; parent ground_link -> ground_step_link
